File: src/kicad/WhimsyCam_KiCad.kicad_sch (KiCad schematic)
At the start: 0 parts

Commit message: made schematic
Parts:
- added J1: GC9A01 Circular Display, symbol Connector_Generic:Conn_01x08
- added SW1: SW_Push, symbol Switch:SW_Push
- added U1: ESP32-S3-WROOM-1, RF_Module:ESP32-S3-WROOM-1, symbol RF_Module:ESP32-S3-WROOM-1
- added U2: ESP32 CAM, symbol Cam:ESP32-cam
Connections:
- new net +3V3: J1.2 (VCC), J1.8 (BLK), U1.2 (3V3)
- new net CS: J1.7 (CS), U1.9 (IO16)
- new net DC: J1.6 (DC), U1.5 (IO5)
- new net GND: J1.1 (GND), SW1.2, U1.1 (GND), U1.40 (GND), U1.41 (GND)
- new net GPIO2: SW1.1, U1.38 (IO2)
- new net RES: J1.5 (RES), U1.4 (IO4)
- new net SCL: J1.3 (SCL), U1.11 (IO18)
- new net SDA: J1.4 (SDA), U1.10 (IO17)
Other:
- note added: "ESP32 S3"
- note added: "TACTILE BUTTON"

Commit message: bom and cad
Parts:
- added J2: TP4056, symbol Connector_Generic:Conn_01x04
Changed lines of the file:
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@@
+	)
+	(symbol
+		(lib_id "Connector_Generic:Conn_01x04")
+		(at 190.5 132.08 90)
+		(unit 1)
+		(exclude_from_sim no)
+		(in_bom yes)
+		(on_board yes)
+		(dnp no)
+		(property "Reference" "J2"
+			(at 190.754 121.412 90)
+			(effects
+				(font
+					(size 1.27 1.27)
+				)
+			)
+		)
+		(property "Value" "TP4056"
+			(at 191.008 123.19 90)
+			(effects
+				(font
+					(size 1.27 1.27)
+				)
+			)
+		)
+		(property "Footprint" ""
+			(at 190.5 132.08 0)
+			(effects
+				(font
+					(size 1.27 1.27)
+				)
+				(hide yes)
+			)
+		)
+		(property "Datasheet" "~"
+			(at 190.5 132.08 0)
+			(effects
+				(font
+					(size 1.27 1.27)
+				)
+				(hide yes)
+			)
+		)
+		(property "Description" "Generic connector, single row, 01x04, script generated (kicad-library-utils/schlib/autogen/connector/)"
+			(at 190.5 132.08 0)
+			(effects
+				(font
+					(size 1.27 1.27)
+				)
+				(hide yes)
+			)
+		)
+		(pin "1"
+		)
+		(pin "3"
+		)
+		(pin "2"
+		)
+		(pin "4"
+		)
+		(instances
+			(project ""
+				(path "/91e2fc71-c974-4ed2-a69d-d8896df8a9cc"
+					(reference "J2")
+					(unit 1)
+				)
+			)
+		)
 	)
 	(symbol
